File: dexter-keypad/dexter-keypad.kicad_sch (KiCad schematic)
At the start: 9 parts, among them J1 Conn_01x07, SW1 SW_Push, SW2 SW_Push, SW3 SW_Push, SW4 RotaryEncoder_Switch_MP, U2 Waveshare ESP32-S3-ZERO

Commit message: feat: polish schematic, create & finish pcb, add gerbers
Parts:
- J1: footprint (none) -> libdexter:Capacitive_Keys
- SW1, SW2, SW3: footprint (none) -> Hackclub Footprints:Kailh Choc Low-Profile Switches
- SW4: footprint (none) -> Rotary_Encoder:RotaryEncoder_Alps_EC11E-Switch_Vertical_H20mm
Connections:
- net ENC1_A: now also U2.2 (GP2); no longer U2.8 (GP8)
- net ENC1_B: now also U2.5 (GP5); no longer U2.9 (GP9)
- net GND: now also SW4.S2
- net LED: now also D3.2 (DIN), U2.3 (GP3); no longer D1.2 (DIN), U2.10 (GP10)
- net SWITCH3: now also U2.1 (GP1); no longer U2.13 (GP13)
- net TOUCH1: now also U2.13 (GP13); no longer U2.1 (GP1)
- net TOUCH2: now also U2.12 (GP12); no longer U2.2 (GP2)
- net TOUCH3: now also U2.11 (GP11); no longer U2.3 (GP3)
- net TOUCH4: now also U2.10 (GP10); no longer U2.4 (GP4)
- net TOUCH5: now also U2.9 (GP9); no longer U2.5 (GP5)
- net TOUCH6: now also U2.8 (GP8); no longer U2.6 (GP6)
- net at D1.4 (DOUT): no longer D2.2 (DIN)
- net at D2.4 (DOUT): now also D1.2 (DIN); no longer D3.2 (DIN)
- net at D3.4 (DOUT): now also D2.2 (DIN)
- net SWITCH_RENCODER: now reaches SW4.S1
- net SWITCH_RENCODER: now also U2.4 (GP4)
Other:
- moved on the sheet: D1
